Commit message: modify urdf from igvc2023 to igvc

File: igvc/urdf/orange.xacro (robot description, xacro)
@@ -16,27 +16,27 @@
   </xacro:macro>
   <!-- Import gazebo reference -->
-  <xacro:include filename="$(find igvc2023)/urdf/orange.gazebo"/>
+  <xacro:include filename="$(find igvc)/urdf/orange.gazebo"/>
   <!-- Import 2D LiDAR model -->
-  <xacro:include filename="$(find igvc2023)/urdf/sensors/hokuyo.urdf.xacro"/>
+  <xacro:include filename="$(find igvc)/urdf/sensors/hokuyo.urdf.xacro"/>
   <xacro:sensor_hokuyo name="hokuyo" parent="base_link" min_angle="-1.22" max_angle="1.22" samples="720">
     <origin xyz="0.16 0.0 0.05" rpy="0.0 0.0 0.0"/>
   </xacro:sensor_hokuyo>
   <!-- Import 3D LiDAR model -->
-  <xacro:include filename="$(find igvc2023)/urdf/sensors/velodyne.urdf.xacro"/>
+  <xacro:include filename="$(find igvc)/urdf/sensors/velodyne.urdf.xacro"/>
   <xacro:sensor_velodyne name="velodyne" parent="base_link" min_angle="-2.35619" max_angle="2.35619" samples="720">
     <origin xyz="-0.13 0.0 0.70" rpy="0.0 0.0 0.0"/>
   </xacro:sensor_velodyne>
   <!-- Import imu model -->
-  <xacro:include filename="$(find igvc2023)/urdf/sensors/imu.urdf.xacro"/>
+  <xacro:include filename="$(find igvc)/urdf/sensors/imu.urdf.xacro"/>
   <xacro:sensor_imu name="imu" parent="base_link" size="0.05 0.05 0.05">
     <origin xyz="0 0.0 0.068" rpy="0.0 0.0 0.0"/>
   </xacro:sensor_imu>
   <!-- Import fisheye camera model -->
-  <xacro:include filename="$(find igvc2023)/urdf/sensors/camera.urdf.xacro"/>
+  <xacro:include filename="$(find igvc)/urdf/sensors/camera.urdf.xacro"/>
   <xacro:sensor_camera name="camera" parent="base_link">
     <origin xyz="-0.13 0 1" rpy="0 0 0"/>
   </xacro:sensor_camera>
   <!-- Import gps model -->
-  <xacro:include filename="$(find igvc2023)/urdf/sensors/gps.urdf.xacro"/>
+  <xacro:include filename="$(find igvc)/urdf/sensors/gps.urdf.xacro"/>
   <xacro:sensor_gps name="gps" parent="base_link">
     <origin xyz="0.5 0 0.75" rpy="0 ${PI} 0"/>
@@ -60,5 +60,5 @@
       <origin xyz="-0.355 0.0 0.3" rpy="0.0 0.0 0.0"/>
       <geometry>
-        <mesh filename="package://igvc2023/meshes/IGVCchassis.dae"/>
+        <mesh filename="package://igvc/meshes/IGVCchassis.dae"/>
       </geometry>
     </visual>
@@ -90,5 +90,5 @@
       <origin xyz="-0.735 0.10 -0.039" rpy="0.0 0.0 0.0"/>
       <geometry>
-        <mesh filename="package://igvc2023/meshes/left_back_wheel.dae"/>
+        <mesh filename="package://igvc/meshes/left_back_wheel.dae"/>
       </geometry>
     </visual>
@@ -104,5 +104,5 @@
       <origin xyz="-0.735 -0.10 -0.039" rpy="0.0 0.0 0.0"/>
       <geometry>
-        <mesh filename="package://igvc2023/meshes/right_back_wheel.dae"/>
+        <mesh filename="package://igvc/meshes/right_back_wheel.dae"/>
         <sphere radius="0.0625"/>
       </geometry>
@@ -134,5 +134,5 @@
       <origin xyz="0.0 0.0 0.0" rpy="0.0 0.0 0.0"/>
       <geometry>
-        <mesh filename="package://igvc2023/meshes/front_wheel.dae"/>
+        <mesh filename="package://igvc/meshes/front_wheel.dae"/>
       </geometry>
     </visual>
@@ -153,5 +153,5 @@
       <origin xyz="0.0 0.0 0.0" rpy="0.0 0.0 0.0"/>
       <geometry>
-        <mesh filename="package://igvc2023/meshes/front_wheel.dae"/>
+        <mesh filename="package://igvc/meshes/front_wheel.dae"/>
       </geometry>
     </visual>

File: igvc/urdf/sensors/hokuyo.urdf.xacro (robot description, xacro)
@@ -21,5 +21,5 @@
         <origin xyz="0 0 0" rpy="0 0 0"/>
         <geometry>
-          <mesh filename="package://igvc2023/meshes/hokuyo.dae"/>
+          <mesh filename="package://igvc/meshes/hokuyo.dae"/>
         </geometry>
       </visual>

File: igvc/urdf/sensors/velodyne.urdf.xacro (robot description, xacro)
@@ -21,5 +21,5 @@
         <origin xyz="0 0 0" rpy="0 0 0"/>
         <geometry>
-          <mesh filename="package://igvc2023/meshes/velodyne.dae"/>
+          <mesh filename="package://igvc/meshes/velodyne.dae"/>
         </geometry>
       </visual>
